Commit message: Added launch files for simulator with and without bullet

File: robots/fetch_fake_base.urdf (robot description, URDF)
Before this commit: robot fetch, 29 links, 28 joints
Links:
- removed link footprint_y
Joints:
- removed joint planar_y_joint
- joint base_turn_joint: child base_link -> footprint_x; parent footprint_y -> odom
- joint planar_x_joint: child footprint_x -> base_link; parent odom -> footprint_x
