Commit message: New URDF and fake controllers. Got rid of opt_test compilation

File: robots/fetch.urdf (robot description, URDF)
Before this commit: robot fetch, 26 links, 25 joints
Links:
- added link fake_gripper_link
Joints:
- added joint gripper_joint: type prismatic, parent gripper_link, child fake_gripper_link, origin xyz=0 0 0 rpy=0 0 0, axis 0 0 1, limit lower=0.0 upper=0.1 effort=60 velocity=0.1

Commit message: Added fake base link for collisions to deal with bullet's odd multibody indices

File: robots/fetch.urdf (robot description, URDF)
Before this commit: robot fetch, 27 links, 26 joints
Links:
- added link base_collision_link, mass 70.1294; collision mesh filename=package://fetch_description/meshes/base_link_collision.STL; visual mesh filename=package://fetch_description/meshes/base_link.dae
- link base_link: mass 70.1294 -> None; geometry 
Joints:
- added joint base_collision_joint: type fixed, parent base_link, child base_collision_link, origin xyz=0 0 0 rpy=0 0 0, axis 0 1 0
- joint l_gripper_finger_joint: mimic (none) -> joint=gripper_joint multiplier=0.5
- joint r_gripper_finger_joint: mimic (none) -> joint=gripper_joint multiplier=0.5
