Commit message: Set torso lift limit to keep it from crushing things on the base

File: robots/fetch_with_box.urdf (robot description, URDF)
Before this commit: robot fetch, 29 links, 28 joints
Joints:
- joint torso_lift_joint: limit lower=0 upper=0.38615 effort=450.0 velocity=0.1 -> lower=0.1 upper=0.38615 effort=450.0 velocity=0.1

Commit message: Limited head tilt downwards angle

File: robots/fetch_with_box.urdf (robot description, URDF)
Before this commit: robot fetch, 29 links, 28 joints
Joints:
- joint head_tilt_joint: limit lower=-0.76 upper=1.45 effort=0.68 velocity=1.57 -> lower=-0.76 upper=1.0 effort=0.68 velocity=1.57
