Commit message: Fix: increase fetch torso lift joint lower bound

File: fetch_temp.urdf (robot description, URDF)
Before this commit: robot fetch, 29 links, 28 joints
Joints:
- joint torso_lift_joint: limit lower=0.0 upper=0.38615 effort=450.0 velocity=0.1 -> lower=0.1 upper=0.38615 effort=450.0 velocity=0.1
